Commit message: Updated STL and added model.config file for gazebo sim.

File: Simulation/jebediah/urdf/jebediah.urdf (robot description, URDF)
Before this commit: robot jebediah, 13 links, 12 joints
Links:
- link Coxa_1: mass 0.12410445572477 -> 0.1241
- link Coxa_2: mass 0.124104455718357 -> 0.1241
- link Coxa_3: mass 0.124104457423663 -> 0.1241
- link Coxa_4: mass 0.124104456070875 -> 0.1241
- link Femur: mass 0.158175969006369 -> 0.15818
- link Femur_1: mass 0.158175969008051 -> 0.15818
- link Femur_2: mass 0.158175969006612 -> 0.15818
- link Femur_4: mass 0.158175969007339 -> 0.15818
- link Tibia_1: mass 0.170868331501115 -> 0.17087
- link Tibia_2: mass 0.170868347804751 -> 0.17087
- link Tibia_3: mass 0.170868354393158 -> 0.17087
- link Tibia_4: mass 0.170868331464115 -> 0.17087
- link base_link: mass 0.297355206086086 -> 0.29736
Joints:
- joint Serv_Coxa_4: limit lower=-1.4 upper=1.4 effort=0.9 velocity=5 -> lower=-1.5708 upper=1.5708 effort=0.9 velocity=5; origin xyz=-0.075112 -0.069996 -0.034543 rpy=7.3339E-15 7.4004E-15 -2.3554 -> xyz=-0.085591 -0.080462 -0.0051626 rpy=7.3339E-15 7.4004E-15 -2.3554
- joint Servo_Coxa_1: limit lower=-1.4 upper=1.4 effort=0.9 velocity=5 -> lower=-1.5708 upper=1.5708 effort=0.9 velocity=5; origin xyz=0.064888 -0.069996 -0.034543 rpy=7.3215E-15 -7.4127E-15 -0.78456 -> xyz=0.075353 -0.080475 -0.0051626 rpy=7.3215E-15 -7.4127E-15 -0.78456
- joint Servo_Coxa_2: limit lower=-1.4 upper=1.4 effort=0.9 velocity=5 -> lower=-1.5708 upper=1.5708 effort=0.9 velocity=5; origin xyz=0.064888 0.070004 -0.034543 rpy=-7.4916E-15 -7.4004E-15 0.78623 -> xyz=0.075367 0.08047 -0.0051626 rpy=-7.4916E-15 -7.4004E-15 0.78623
- joint Servo_Coxa_3: limit lower=-1.4 upper=1.4 effort=0.9 velocity=5 -> lower=-1.5708 upper=1.5708 effort=0.9 velocity=5; origin xyz=-0.075112 0.070004 -0.034543 rpy=-7.4792E-15 7.4127E-15 2.357 -> xyz=-0.085578 0.080483 -0.0051626 rpy=-7.4792E-15 7.4127E-15 2.357
- joint Servo_Femur_1_1: limit lower=-1.4 upper=1.4 effort=0.9 velocity=5 -> lower=-1.5708 upper=1.5708 effort=0.9 velocity=5; origin xyz=0.064665 -0.028419 0.029 rpy=-1.3192E-16 -2.7756E-17 -2.7756E-16 -> xyz=0.10132 -0.0015074 -0.00036453 rpy=-1.3192E-16 -2.7756E-17 -2.7756E-16
- joint Servo_Femur_1_2: limit lower=-1.4 upper=1.4 effort=0.9 velocity=5 -> lower=-1.5708 upper=1.5708 effort=0.9 velocity=5; origin xyz=0.10294 0.028419 0 rpy=8.3049E-16 2.7756E-17 5.3294E-29 -> xyz=0.069261 0.0014932 -0.04833 rpy=8.3049E-16 2.7756E-17 5.3294E-29
- joint Servo_Femur_2_1: axis 0 -1 0 -> 0 1 0; limit lower=-1.4 upper=1.4 effort=0.9 velocity=5 -> lower=-1.5708 upper=1.5708 effort=0.9 velocity=5; origin xyz=0.064665 -0.028419 0.029 rpy=-1.3192E-16 -2.7756E-17 -3.3307E-16 -> xyz=0.10132 -0.0015074 -0.00036453 rpy=-1.3192E-16 -2.7756E-17 -3.3307E-16
- joint Servo_Femur_2_2: axis 0 -1 0 -> 0 1 0; limit lower=-1.4 upper=1.4 effort=0.9 velocity=5 -> lower=-1.5708 upper=1.5708 effort=0.9 velocity=0; origin xyz=0.10294 0.028419 0 rpy=8.3049E-16 2.7756E-17 -5.6417E-29 -> xyz=0.069261 0.0014932 -0.04833 rpy=8.3049E-16 2.7756E-17 -5.6417E-29
- joint Servo_Femur_3_1: axis 0 -1 0 -> 0 1 0; limit lower=-1.4 upper=1.4 effort=0.9 velocity=5 -> lower=-1.5708 upper=1.5708 effort=0.9 velocity=5; origin xyz=0.064665 -0.028419 0.029 rpy=-1.3192E-16 -2.7756E-17 -3.3307E-16 -> xyz=0.10132 -0.0015074 -0.00036453 rpy=-1.3192E-16 -2.7756E-17 -3.3307E-16
- joint Servo_Femur_3_2: axis 0 -1 0 -> 0 1 0; limit lower=-1.4 upper=1.4 effort=0.9 velocity=5 -> lower=-1.5708 upper=1.5708 effort=0.9 velocity=5; origin xyz=0.10294 0.028419 0 rpy=8.3049E-16 2.7756E-17 5.6419E-29 -> xyz=0.069261 0.0014932 -0.04833 rpy=8.3049E-16 2.7756E-17 5.6419E-29
- joint Servo_Femur_4_1: limit lower=-1.4 upper=1.4 effort=0.9 velocity=5 -> lower=-1.5708 upper=1.5708 effort=0.9 velocity=5; origin xyz=0.064665 -0.028419 0.029 rpy=-1.3192E-16 -2.7756E-17 -2.7756E-16 -> xyz=0.10132 -0.0015074 -0.00036453 rpy=-1.3192E-16 -2.7756E-17 -2.7756E-16
- joint Servo_Femur_4_2: limit lower=-1.4 upper=1.4 effort=0.9 velocity=5 -> lower=-1.5708 upper=1.5708 effort=0.9 velocity=5; origin xyz=0.10294 0.028419 0 rpy=8.3049E-16 2.7756E-17 -5.3297E-29 -> xyz=0.069261 0.0014932 -0.04833 rpy=8.3049E-16 2.7756E-17 -5.3297E-29

Commit message: Re-up simulation files.

File: Simulation/jebediah/urdf/jebediah.urdf (robot description, URDF)
Before this commit: robot jebediah, 13 links, 12 joints
Links:
- link Coxa_1: mass 0.1241 -> 0.12410445572477
- link Coxa_2: mass 0.1241 -> 0.124104455718357
- link Coxa_3: mass 0.1241 -> 0.124104457423663
- link Coxa_4: mass 0.1241 -> 0.124104456070875
- link Femur: mass 0.15818 -> 0.158175969006369
- link Femur_1: mass 0.15818 -> 0.158175969008051
- link Femur_2: mass 0.15818 -> 0.158175969006612
- link Femur_4: mass 0.15818 -> 0.158175969007339
- link Tibia_1: mass 0.17087 -> 0.170868331501115
- link Tibia_2: mass 0.17087 -> 0.170868347804751
- link Tibia_3: mass 0.17087 -> 0.170868354393158
- link Tibia_4: mass 0.17087 -> 0.170868331464115
- link base_link: mass 0.29736 -> 0.297355206086086
Joints:
- joint Serv_Coxa_4: limit lower=-1.5708 upper=1.5708 effort=0.9 velocity=5 -> lower=-1.4 upper=1.4 effort=0.9 velocity=5; origin xyz=-0.085591 -0.080462 -0.0051626 rpy=7.3339E-15 7.4004E-15 -2.3554 -> xyz=-0.075112 -0.069996 -0.034543 rpy=7.3339E-15 7.4004E-15 -2.3554
- joint Servo_Coxa_1: limit lower=-1.5708 upper=1.5708 effort=0.9 velocity=5 -> lower=-1.4 upper=1.4 effort=0.9 velocity=5; origin xyz=0.075353 -0.080475 -0.0051626 rpy=7.3215E-15 -7.4127E-15 -0.78456 -> xyz=0.064888 -0.069996 -0.034543 rpy=7.3215E-15 -7.4127E-15 -0.78456
- joint Servo_Coxa_2: limit lower=-1.5708 upper=1.5708 effort=0.9 velocity=5 -> lower=-1.4 upper=1.4 effort=0.9 velocity=5; origin xyz=0.075367 0.08047 -0.0051626 rpy=-7.4916E-15 -7.4004E-15 0.78623 -> xyz=0.064888 0.070004 -0.034543 rpy=-7.4916E-15 -7.4004E-15 0.78623
- joint Servo_Coxa_3: limit lower=-1.5708 upper=1.5708 effort=0.9 velocity=5 -> lower=-1.4 upper=1.4 effort=0.9 velocity=5; origin xyz=-0.085578 0.080483 -0.0051626 rpy=-7.4792E-15 7.4127E-15 2.357 -> xyz=-0.075112 0.070004 -0.034543 rpy=-7.4792E-15 7.4127E-15 2.357
- joint Servo_Femur_1_1: limit lower=-1.5708 upper=1.5708 effort=0.9 velocity=5 -> lower=-1.4 upper=1.4 effort=0.9 velocity=5; origin xyz=0.10132 -0.0015074 -0.00036453 rpy=-1.3192E-16 -2.7756E-17 -2.7756E-16 -> xyz=0.064665 -0.028419 0.029 rpy=-1.3192E-16 -2.7756E-17 -2.7756E-16
- joint Servo_Femur_1_2: limit lower=-1.5708 upper=1.5708 effort=0.9 velocity=5 -> lower=-1.4 upper=1.4 effort=0.9 velocity=5; origin xyz=0.069261 0.0014932 -0.04833 rpy=8.3049E-16 2.7756E-17 5.3294E-29 -> xyz=0.10294 0.028419 0 rpy=8.3049E-16 2.7756E-17 5.3294E-29
- joint Servo_Femur_2_1: axis 0 1 0 -> 0 -1 0; limit lower=-1.5708 upper=1.5708 effort=0.9 velocity=5 -> lower=-1.4 upper=1.4 effort=0.9 velocity=5; origin xyz=0.10132 -0.0015074 -0.00036453 rpy=-1.3192E-16 -2.7756E-17 -3.3307E-16 -> xyz=0.064665 -0.028419 0.029 rpy=-1.3192E-16 -2.7756E-17 -3.3307E-16
- joint Servo_Femur_2_2: axis 0 1 0 -> 0 -1 0; limit lower=-1.5708 upper=1.5708 effort=0.9 velocity=0 -> lower=-1.4 upper=1.4 effort=0.9 velocity=5; origin xyz=0.069261 0.0014932 -0.04833 rpy=8.3049E-16 2.7756E-17 -5.6417E-29 -> xyz=0.10294 0.028419 0 rpy=8.3049E-16 2.7756E-17 -5.6417E-29
- joint Servo_Femur_3_1: axis 0 1 0 -> 0 -1 0; limit lower=-1.5708 upper=1.5708 effort=0.9 velocity=5 -> lower=-1.4 upper=1.4 effort=0.9 velocity=5; origin xyz=0.10132 -0.0015074 -0.00036453 rpy=-1.3192E-16 -2.7756E-17 -3.3307E-16 -> xyz=0.064665 -0.028419 0.029 rpy=-1.3192E-16 -2.7756E-17 -3.3307E-16
- joint Servo_Femur_3_2: axis 0 1 0 -> 0 -1 0; limit lower=-1.5708 upper=1.5708 effort=0.9 velocity=5 -> lower=-1.4 upper=1.4 effort=0.9 velocity=5; origin xyz=0.069261 0.0014932 -0.04833 rpy=8.3049E-16 2.7756E-17 5.6419E-29 -> xyz=0.10294 0.028419 0 rpy=8.3049E-16 2.7756E-17 5.6419E-29
- joint Servo_Femur_4_1: limit lower=-1.5708 upper=1.5708 effort=0.9 velocity=5 -> lower=-1.4 upper=1.4 effort=0.9 velocity=5; origin xyz=0.10132 -0.0015074 -0.00036453 rpy=-1.3192E-16 -2.7756E-17 -2.7756E-16 -> xyz=0.064665 -0.028419 0.029 rpy=-1.3192E-16 -2.7756E-17 -2.7756E-16
- joint Servo_Femur_4_2: limit lower=-1.5708 upper=1.5708 effort=0.9 velocity=5 -> lower=-1.4 upper=1.4 effort=0.9 velocity=5; origin xyz=0.069261 0.0014932 -0.04833 rpy=8.3049E-16 2.7756E-17 -5.3297E-29 -> xyz=0.10294 0.028419 0 rpy=8.3049E-16 2.7756E-17 -5.3297E-29
